File: Programer/Nano AT85 programer/Nano AT85 programer.kicad_sch (KiCad schematic)
At the start: 4 parts, among them U1 ATtiny85V-10P

Commit message: Values added
Parts:
- C1: value C -> 100n (104)
- C2: value C_Polarized -> 10uF
Changed lines of the file:
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@@
   )
   (symbol (lib_id "Device:C") (at 64.77 106.68 0) (unit 1)
-    (in_bom yes) (on_board yes) (fields_autoplaced)
+    (in_bom yes) (on_board yes)
     (property "Reference" "C1" (id 0) (at 68.58 105.4099 0)
       (effects (font (size 1.27 1.27)) (justify left))
     )
-    (property "Value" "C" (id 1) (at 68.58 107.9499 0)
+    (property "Value" "100n (104)" (id 1) (at 58.42 110.49 0)
       (effects (font (size 1.27 1.27)) (justify left))
     )
@@
       (effects (font (size 1.27 1.27)) (justify left))
     )
-    (property "Value" "C_Polarized" (id 1) (at 173.99 113.4109 0)
+    (property "Value" "10uF" (id 1) (at 173.99 113.4109 0)
       (effects (font (size 1.27 1.27)) (justify left))
     )
@@
     )
     (path "/a3127a85-1896-404a-897b-30a2206361d4"
-      (reference "C1") (unit 1) (value "C") (footprint "Capacitor_THT:C_Disc_D4.7mm_W2.5mm_P5.00mm")
+      (reference "C1") (unit 1) (value "100n (104)") (footprint "Capacitor_THT:C_Disc_D4.7mm_W2.5mm_P5.00mm")
     )
     (path "/f0543d83-eb30-4cb5-81ee-61ddd1b78eb5"
-      (reference "C2") (unit 1) (value "C_Polarized") (footprint "Capacitor_THT:CP_Radial_D6.3mm_P2.50mm")
+      (reference "C2") (unit 1) (value "10uF") (footprint "Capacitor_THT:CP_Radial_D6.3mm_P2.50mm")
     )
     (path "/ac3034ee-3ed9-41d5-b548-d47a43d4e9c1"
