File: Programer/Nano AT85 programer/Nano AT85 programer.kicad_pcb (KiCad board)
At the start: 2 copper layers, 52.5 x 58.5 mm, 4 parts, among them U1 ATtiny85V-10P

Commit message: stuff git push
git stsatu

git status
''jjj
Parts:
- C1: value C -> 100n (104)
- C2: value C_Polarized -> 10uF
Changed lines of the file:
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@@
       (effects (font (size 1 1) (thickness 0.15)))
     )
-    (fp_text value "C" (at 2.5 2.5) (layer "F.Fab")
+    (fp_text value "100n (104)" (at 2.5 2.5) (layer "F.Fab")
       (effects (font (size 1 1) (thickness 0.15)))
     )
@@
       (effects (font (size 1 1) (thickness 0.15)))
     )
-    (fp_text value "C_Polarized" (at 1.25 4.4) (layer "F.Fab")
+    (fp_text value "10uF" (at 1.25 4.4) (layer "F.Fab")
       (effects (font (size 1 1) (thickness 0.15)))
     )
